File: letThereBeLight.kicad_pcb (KiCad board)
At the start: 2 copper layers, 0 parts

Commit message: generate gerber files
Parts:
- added BT1: 3.3V Cell, Battery:BatteryHolder_ComfortableElectronic_CH273-2450_1x2450, F.Cu at (124.0, 100.0)
- added D1: 5mm Yellow LED, LED_THT:LED_D5.0mm, F.Cu at (159.0, 102.0)
- added MK1: Microphone_Condenser, Connector_PinHeader_2.54mm:PinHeader_1x02_P2.54mm_Vertical, F.Cu at (175.0, 99.5)
- added R1: 10k, Resistor_THT:R_Axial_DIN0207_L6.3mm_D2.5mm_P15.24mm_Horizontal, F.Cu at (154.8, 81.5)
- added R2: 5mm LDR, OptoDevice:R_LDR_5.1x4.3mm_P3.4mm_Vertical, F.Cu at (168.0, 102.5)
- added R3: 5.6k, Resistor_THT:R_Axial_DIN0207_L6.3mm_D2.5mm_P15.24mm_Horizontal, F.Cu at (154.8, 86.2)
- added R4: 470R, Resistor_THT:R_Axial_DIN0207_L6.3mm_D2.5mm_P15.24mm_Horizontal, F.Cu at (154.8, 91.0)
- added SW2: SW_SPDT, Button_Switch_THT:SW_Slide_SPDT_Angled_CK_OS102011MA1Q, F.Cu at (145.1, 119.5)
- added U1: ATtiny85V-10P, Package_DIP:DIP-8_W7.62mm, F.Cu at (158.9, 118.6)
Routing:
- net GND: track 0.00 -> 81.2 mm
- net +3.3V: track 0.00 -> 79.3 mm
- net /LDR: track 0.00 -> 44.0 mm
- net /MIC: track 0.00 -> 42.4 mm
- net Net-(BT1--): track 0.00 -> 21.4 mm
- net Net-(D1-K): track 0.00 -> 13.4 mm
- added copper zone on B.Cu, net GND
- added copper zone on F.Cu, net GND
Other:
- board outline added: 60 x 60 mm
- board text added: "ABR"
