File: letThereBeLight.kicad_sch (KiCad schematic)
At the start: 9 parts, among them SW2 SW_SPDT, U1 ATtiny85V-10P

Commit message: generate gerber files
Connections:
- net LED: no longer D1.1 (K), R4.1
- new net: D1.1 (K), R4.1
Other:
- moved on the sheet: SW2
Changed lines of the file:
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@@
 	)
 	(junction
-		(at 224.79 95.25)
+		(at 68.58 109.22)
 		(diameter 0)
 		(color 0 0 0 0)
 	)
 	(junction
-		(at 68.58 109.22)
+		(at 68.58 104.14)
 		(diameter 0)
 		(color 0 0 0 0)
@@
 	)
 	(no_connect
-		(at 66.04 91.44)
+		(at 66.04 93.98)
 	)
 	(no_connect
@@
 	(wire
 		(pts
-			(xy 224.79 95.25) (xy 234.95 95.25)
-		)
-		(stroke
-			(width 0)
-			(type default)
-		)
-	)
-	(wire
-		(pts
 			(xy 71.12 82.55) (xy 81.28 82.55)
 		)
@@
 	(wire
 		(pts
-			(xy 224.79 91.44) (xy 224.79 95.25)
+			(xy 162.56 93.98) (xy 162.56 96.52)
 		)
 		(stroke
@@
 	(wire
 		(pts
-			(xy 162.56 93.98) (xy 162.56 96.52)
+			(xy 190.5 93.98) (xy 190.5 96.52)
 		)
 		(stroke
@@
 	(wire
 		(pts
-			(xy 190.5 93.98) (xy 190.5 96.52)
+			(xy 224.79 104.14) (xy 224.79 111.76)
 		)
 		(stroke
@@
 	(wire
 		(pts
-			(xy 224.79 104.14) (xy 224.79 111.76)
+			(xy 224.79 91.44) (xy 224.79 96.52)
 		)
 		(stroke
@@
 	(wire
 		(pts
-			(xy 224.79 95.25) (xy 224.79 96.52)
+			(xy 190.5 91.44) (xy 190.5 93.98)
 		)
 		(stroke
@@
 	(wire
 		(pts
-			(xy 190.5 91.44) (xy 190.5 93.98)
+			(xy 71.12 91.44) (xy 71.12 93.98)
 		)
 		(stroke
@@
 	(wire
 		(pts
-			(xy 68.58 101.6) (xy 68.58 109.22)
+			(xy 68.58 101.6) (xy 68.58 104.14)
 		)
 		(stroke
@@
 		)
 	)
+	(wire
+		(pts
+			(xy 68.58 104.14) (xy 68.58 109.22)
+		)
+		(stroke
+			(width 0)
+			(type default)
+		)
+	)
 	(image
 		(at 199.39 173.99)
@@
 		)
 	)
-	(label "LED"
-		(at 234.95 95.25 0)
+	(label "LDR"
+		(at 149.86 93.98 0)
 		(effects
 			(font
@@
 		)
 	)
-	(label "LDR"
-		(at 149.86 93.98 0)
+	(label "MIC"
+		(at 140.97 96.52 0)
 		(effects
 			(font
@@
 		)
 	)
-	(label "MIC"
-		(at 140.97 96.52 0)
+	(netclass_flag ""
+		(length 0.0102)
+		(shape dot)
+		(at 71.12 92.71 0)
+		(fields_autoplaced yes)
+		(effects
+			(font
+				(size 1.27 1.27)
+			)
+			(justify left bottom)
+		)
+		(property "Netclass" "signal"
+			(at 71.8185 92.6998 0)
+			(effects
+				(font
+					(size 1.27 1.27)
+				)
+				(justify left)
+				(hide yes)
+			)
+		)
+		(property "Component Class" ""
+			(at -2.54 0 0)
+			(effects
+				(font
+					(size 1.27 1.27)
+					(italic yes)
+				)
+			)
+		)
+	)
+	(netclass_flag ""
+		(length 0.0102)
+		(shape dot)
+		(at 224.79 95.25 0)
+		(fields_autoplaced yes)
 		(effects
 			(font
@@
 			(justify left bottom)
 		)
+		(property "Netclass" "signal"
+			(at 225.4885 95.2398 0)
+			(effects
+				(font
+					(size 1.27 1.27)
+					(italic yes)
+				)
+				(justify left)
+				(hide yes)
+			)
+		)
+		(property "Component Class" ""
+			(at -49.53 6.35 0)
+			(effects
+				(font
+					(size 1.27 1.27)
+					(italic yes)
+				)
+			)
+		)
 	)
 	(symbol
@@
 	(symbol
 		(lib_id "Switch:SW_SPDT")
-		(at 68.58 96.52 90)
+		(at 68.58 99.06 90)
 		(unit 1)
 		(exclude_from_sim no)
@@
 		(fields_autoplaced yes)
 		(property "Reference" "SW2"
-			(at 73.66 95.2499 90)
+			(at 73.66 97.7899 90)
 			(effects
 				(font
@@
 		)
 		(property "Value" "SW_SPDT"
-			(at 73.66 97.7899 90)
+			(at 73.66 100.3299 90)
 			(effects
 				(font
@@
 		)
 		(property "Footprint" "Button_Switch_THT:SW_Slide_SPDT_Angled_CK_OS102011MA1Q"
-			(at 68.58 96.52 0)
+			(at 68.58 99.06 0)
 			(effects
 				(font
@@
 		)
 		(property "Datasheet" "~"
-			(at 76.2 96.52 0)
+			(at 76.2 99.06 0)
 			(effects
 				(font
@@
 		)
 		(property "Description" "Switch, single pole double throw"
-			(at 68.58 96.52 0)
+			(at 68.58 99.06 0)
 			(effects
 				(font
